File: Quiz_Buzzer.sch (KiCad schematic (older format))
At the start: 26 parts, among them J1 Barrel_Jack_Switch, U1 ATmega328P-PU, U2 CD74HC4067M, Y1 Crystal

Commit message: adding all missing components in schematic file
Parts:
- added BZ1: Buzzer, symbol Device:Buzzer
- added R10, R11, R12, R13, R14, R15, R16, R17, R18, R19, R20: 5k, symbol Device:R
- added SW1, SW10, SW11, SW2, SW3, SW4, SW5, SW6, SW7, SW8, SW9: SW_Push_Dual, symbol Switch:SW_Push_Dual
- R2, R3, R4, R5, R6, R7, R8, R9: value R -> 200
Connections:
- wire segments 94 -> 175
Other:
- note added: "Arduino Representation\n"
- moved on the sheet: C1, C2, C3, C4, C5, D5, D6, D7, D8, R6, R7, R8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

Commit message: added pcb layout trial1
Parts:
- BZ1: footprint (none) -> Buzzer_Beeper:Buzzer_12x9.5RM7.6
- C1, C2, C3, C4, C5: footprint (none) -> Capacitor_THT:C_Axial_L3.8mm_D2.6mm_P7.50mm_Horizontal
- D1, D2, D3, D4, D5, D6, D7, D8: footprint (none) -> LED_THT:LED_D3.0mm
- J1: footprint (none) -> Connector_BarrelJack:BarrelJack_CLIFF_FC681465S_SMT_Horizontal
- R1, R10, R11, R12, R13, R14, R15, R16, R17, R18, R19, R2, R20, R3, R4, R5, R6, R7, R8, R9: footprint (none) -> Resistor_THT:R_Axial_DIN0309_L9.0mm_D3.2mm_P12.70mm_Horizontal
- SW1, SW10, SW11, SW2, SW3, SW4, SW5, SW6, SW7, SW8, SW9: footprint (none) -> Button_Switch_THT:SW_PUSH_6mm; symbol Switch:SW_Push_Dual -> Switch:SW_DIP_x01
- Y1: footprint (none) -> Crystal:Crystal_HC49-4H_Vertical
Connections:
- wire segments 175 -> 153
- no-connect marks 0 -> 12
Other:
- note removed: "Arduino Representation\n"
- moved on the sheet: BZ1, D1, D2, D3, D4, D5, D6, D7, D8, J1, R10, R12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

Commit message: Saving current work to make sure I don't lose it
Parts:
- added J?: Conn_01x03_Male, symbol Connector:Conn_01x03_Male
- added J? (x2): Conn_01x04_Male, symbol Connector:Conn_01x04_Male
Connections:
- wire segments 153 -> 168
Changed lines of the file:
@@
 	10400 1450 10550 1450
 Wire Wire Line
-	10450 2850 10600 2850
+	10450 2850 10500 2850
 Wire Wire Line
 	10500 4150 10650 4150
@@
 Wire Wire Line
 	10700 5950 10750 5950
+$Comp
+L Connector:Conn_01x03_Male J?
+U 1 1 61271B78
+P 8150 1900
+F 0 "J?" H 8258 2181 50  0000 C CNN
+F 1 "Conn_01x03_Male" H 8258 2090 50  0000 C CNN
+F 2 "" H 8150 1900 50  0001 C CNN
+F 3 "~" H 8150 1900 50  0001 C CNN
+	1    8150 1900
+	1    0    0    -1
+$EndComp
+$Comp
+L Connector:Conn_01x04_Male J?
+U 1 1 61273571
+P 6950 4900
+F 0 "J?" H 7058 5181 50  0000 C CNN
+F 1 "Conn_01x04_Male" H 7058 5090 50  0000 C CNN
+F 2 "" H 6950 4900 50  0001 C CNN
+F 3 "~" H 6950 4900 50  0001 C CNN
+	1    6950 4900
+	1    0    0    -1
+$EndComp
+Text GLabel 7300 4800 2    50   Input ~ 0
+P12
+Wire Wire Line
+	7150 4800 7300 4800
+$Comp
+L power:GND #PWR?
+U 1 1 6127DBFB
+P 7300 4900
+F 0 "#PWR?" H 7300 4650 50  0001 C CNN
+F 1 "GND" V 7305 4772 50  0000 R CNN
+F 2 "" H 7300 4900 50  0001 C CNN
+F 3 "" H 7300 4900 50  0001 C CNN
+	1    7300 4900
+	0    -1   -1   0
+$EndComp
+Wire Wire Line
+	7150 4900 7300 4900
+Text GLabel 7300 5000 2    50   Input ~ 0
+L12
+$Comp
+L power:+5V #PWR?
+U 1 1 61288FCD
+P 7300 5150
+F 0 "#PWR?" H 7300 5000 50  0001 C CNN
+F 1 "+5V" V 7315 5278 50  0000 L CNN
+F 2 "" H 7300 5150 50  0001 C CNN
+F 3 "" H 7300 5150 50  0001 C CNN
+	1    7300 5150
+	0    1    1    0
+$EndComp
+Wire Wire Line
+	7300 5150 7150 5150
+Wire Wire Line
+	7150 5150 7150 5100
+Wire Wire Line
+	7250 5000 7150 5000
+$Comp
+L Connector:Conn_01x04_Male J?
+U 1 1 612BA812
+P 8950 3250
+F 0 "J?" H 9058 3531 50  0000 C CNN
+F 1 "Conn_01x04_Male" H 9058 3440 50  0000 C CNN
+F 2 "" H 8950 3250 50  0001 C CNN
+F 3 "~" H 8950 3250 50  0001 C CNN
+	1    8950 3250
+	1    0    0    -1
+$EndComp
+$Comp
+L power:+5V #PWR?
+U 1 1 612BA822
+P 9300 3500
+F 0 "#PWR?" H 9300 3350 50  0001 C CNN
+F 1 "+5V" V 9315 3628 50  0000 L CNN
+F 2 "" H 9300 3500 50  0001 C CNN
+F 3 "" H 9300 3500 50  0001 C CNN
+	1    9300 3500
+	0    1    1    0
+$EndComp
+Wire Wire Line
+	9300 3500 9150 3500
+Wire Wire Line
+	9150 3500 9150 3450
+Wire Wire Line
+	9250 3350 9150 3350
+Wire Wire Line
+	10000 3150 10000 3400
+Wire Wire Line
+	10000 3400 10050 3400
+Wire Wire Line
+	10050 3400 10050 3450
+Wire Wire Line
+	9150 3150 10000 3150
+Wire Wire Line
+	10500 3250 10500 2850
+Wire Wire Line
+	9150 3250 10500 3250
+Connection ~ 10500 2850
+Wire Wire Line
+	10500 2850 10600 2850
 $EndSCHEMATC
